File: MotorController.sch (EAGLE design)
At the start: 13 parts

Commit message: pcb design waiting for inspection
Connections:
- removed net 5V: CON1.8, U$6.OUT
- removed net N$14: U$2.EN_N
- removed net N$9: U$1.EN_N
- net GND: now also U$1.EN_N, U$2.EN_N, U$6.IN
- net VBAT: now also U$6.EN; no longer U$6.IN
- net VCC: now also CON1.8, U$6.OUT
Changed lines of the file:
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@@
 <?xml version="1.0" encoding="utf-8"?>
 <!DOCTYPE eagle SYSTEM "eagle.dtd">
-<eagle version="9.5.2">
+<eagle version="9.6.0">
 <drawing>
 <settings>
@@
 <part name="P+1" library="supply1" library_urn="urn:adsk.eagle:library:371" deviceset="VCC" device=""/>
 <part name="P+2" library="supply1" library_urn="urn:adsk.eagle:library:371" deviceset="VCC" device=""/>
-<part name="P+3" library="supply1" library_urn="urn:adsk.eagle:library:371" deviceset="VCC" device=""/>
 <part name="J1" library="SparkFun-Connectors" deviceset="CONN_05" device=""/>
 <part name="J2" library="SparkFun-Connectors" deviceset="CONN_05" device=""/>
@@
 <part name="GND10" library="supply1" library_urn="urn:adsk.eagle:library:371" deviceset="GND" device=""/>
 <part name="J5" library="SparkFun-Connectors" deviceset="CONN_02" device="5MM"/>
+<part name="GND5" library="supply1" library_urn="urn:adsk.eagle:library:371" deviceset="GND" device=""/>
+<part name="P+3" library="supply1" library_urn="urn:adsk.eagle:library:371" deviceset="VCC" device=""/>
+<part name="P+4" library="supply1" library_urn="urn:adsk.eagle:library:371" deviceset="VCC" device=""/>
+<part name="GND7" library="supply1" library_urn="urn:adsk.eagle:library:371" deviceset="GND" device=""/>
+<part name="GND11" library="supply1" library_urn="urn:adsk.eagle:library:371" deviceset="GND" device=""/>
 </parts>
 <sheets>
@@
 <attribute name="VALUE" x="96.52" y="152.4" size="1.778" layer="96" rot="R90"/>
 </instance>
-<instance part="P+3" gate="VCC" x="177.8" y="193.04" smashed="yes">
-<attribute name="VALUE" x="175.26" y="190.5" size="1.778" layer="96" rot="R90"/>
-</instance>
 <instance part="J1" gate="G$1" x="210.82" y="167.64" smashed="yes" rot="R180">
 <attribute name="VALUE" x="213.36" y="177.546" size="1.778" layer="96" font="vector" rot="R180"/>
@@
 <attribute name="VALUE" x="27.94" y="112.014" size="1.778" layer="96" font="vector"/>
 <attribute name="NAME" x="27.94" y="122.428" size="1.778" layer="95" font="vector"/>
+</instance>
+<instance part="GND5" gate="1" x="187.96" y="109.22" smashed="yes">
+<attribute name="VALUE" x="185.42" y="106.68" size="1.778" layer="96"/>
+</instance>
+<instance part="P+3" gate="VCC" x="180.34" y="111.76" smashed="yes" rot="MR0">
+<attribute name="VALUE" x="182.88" y="109.22" size="1.778" layer="96" rot="MR90"/>
+</instance>
+<instance part="P+4" gate="VCC" x="22.86" y="185.42" smashed="yes">
+<attribute name="VALUE" x="20.32" y="182.88" size="1.778" layer="96" rot="R90"/>
+</instance>
+<instance part="GND7" gate="1" x="116.84" y="185.42" smashed="yes">
+<attribute name="VALUE" x="114.3" y="182.88" size="1.778" layer="96"/>
+</instance>
+<instance part="GND11" gate="1" x="114.3" y="152.4" smashed="yes">
+<attribute name="VALUE" x="111.76" y="149.86" size="1.778" layer="96"/>
 </instance>
 </instances>
@@
 </segment>
 <segment>
-<pinref part="U$6" gate="G$1" pin="GND"/>
-<wire x1="203.2" y1="111.76" x2="193.04" y2="111.76" width="0.1524" layer="91"/>
-<label x="193.04" y="111.76" size="1.778" layer="95"/>
-</segment>
-<segment>
 <pinref part="C3" gate="G$1" pin="-"/>
 <pinref part="GND9" gate="1" pin="GND"/>
@@
 <wire x1="40.64" y1="116.84" x2="38.1" y2="116.84" width="0.1524" layer="91"/>
 </segment>
-</net>
-<net name="5V" class="0">
-<segment>
-<pinref part="CON1" gate="G$1" pin="8"/>
-<wire x1="35.56" y1="180.34" x2="27.94" y2="180.34" width="0.1524" layer="91"/>
-<label x="27.94" y="180.34" size="1.778" layer="95"/>
-</segment>
-<segment>
-<pinref part="P+3" gate="VCC" pin="VCC"/>
-<wire x1="177.8" y1="190.5" x2="177.8" y2="187.96" width="0.1524" layer="91"/>
-<wire x1="177.8" y1="187.96" x2="182.88" y2="187.96" width="0.1524" layer="91"/>
-<label x="180.34" y="187.96" size="1.778" layer="95"/>
-</segment>
-<segment>
-<pinref part="U$6" gate="G$1" pin="OUT"/>
-<wire x1="203.2" y1="106.68" x2="193.04" y2="106.68" width="0.1524" layer="91"/>
-<label x="193.04" y="106.68" size="1.778" layer="95"/>
+<segment>
+<pinref part="U$6" gate="G$1" pin="IN"/>
+<wire x1="203.2" y1="116.84" x2="187.96" y2="116.84" width="0.1524" layer="91"/>
+<pinref part="GND5" gate="1" pin="GND"/>
+<wire x1="187.96" y1="116.84" x2="187.96" y2="111.76" width="0.1524" layer="91"/>
+<pinref part="U$6" gate="G$1" pin="GND"/>
+<wire x1="203.2" y1="111.76" x2="187.96" y2="111.76" width="0.1524" layer="91"/>
+<junction x="187.96" y="111.76"/>
+</segment>
+<segment>
+<pinref part="U$1" gate="G$1" pin="EN_N"/>
+<wire x1="121.92" y1="180.34" x2="124.46" y2="180.34" width="0.1524" layer="91"/>
+<wire x1="121.92" y1="180.34" x2="121.92" y2="187.96" width="0.1524" layer="91"/>
+<wire x1="121.92" y1="187.96" x2="116.84" y2="187.96" width="0.1524" layer="91"/>
+<pinref part="GND7" gate="1" pin="GND"/>
+</segment>
+<segment>
+<pinref part="U$2" gate="G$1" pin="EN_N"/>
+<wire x1="124.46" y1="147.32" x2="119.38" y2="147.32" width="0.1524" layer="91"/>
+<wire x1="119.38" y1="147.32" x2="119.38" y2="154.94" width="0.1524" layer="91"/>
+<pinref part="GND11" gate="1" pin="GND"/>
+<wire x1="119.38" y1="154.94" x2="114.3" y2="154.94" width="0.1524" layer="91"/>
 </segment>
 </net>
@@
 </segment>
 <segment>
-<pinref part="U$6" gate="G$1" pin="IN"/>
-<wire x1="203.2" y1="116.84" x2="193.04" y2="116.84" width="0.1524" layer="91"/>
-<label x="193.04" y="116.84" size="1.778" layer="95"/>
+<pinref part="U$6" gate="G$1" pin="EN"/>
+<wire x1="203.2" y1="121.92" x2="193.04" y2="121.92" width="0.1524" layer="91"/>
+<label x="193.04" y="121.92" size="1.778" layer="95"/>
 </segment>
 </net>
@@
 <wire x1="152.4" y1="147.32" x2="157.48" y2="147.32" width="0.1524" layer="91"/>
 <label x="157.48" y="147.32" size="1.778" layer="95"/>
-</segment>
-</net>
-<net name="N$9" class="0">
-<segment>
-<pinref part="U$1" gate="G$1" pin="EN_N"/>
-<wire x1="121.92" y1="180.34" x2="124.46" y2="180.34" width="0.1524" layer="91"/>
-</segment>
-</net>
-<net name="N$14" class="0">
-<segment>
-<pinref part="U$2" gate="G$1" pin="EN_N"/>
-<wire x1="121.92" y1="147.32" x2="124.46" y2="147.32" width="0.1524" layer="91"/>
 </segment>
 </net>
@@
 <wire x1="96.52" y1="134.62" x2="96.52" y2="149.86" width="0.1524" layer="91"/>
 </segment>
-</net>
+<segment>
+<pinref part="U$6" gate="G$1" pin="OUT"/>
+<label x="193.04" y="106.68" size="1.778" layer="95"/>
+<pinref part="P+3" gate="VCC" pin="VCC"/>
+<wire x1="203.2" y1="106.68" x2="195.58" y2="106.68" width="0.1524" layer="91"/>
+<wire x1="193.04" y1="106.68" x2="180.34" y2="106.68" width="0.1524" layer="91"/>
+<wire x1="180.34" y1="106.68" x2="180.34" y2="109.22" width="0.1524" layer="91"/>
+<wire x1="195.58" y1="106.68" x2="193.04" y2="106.68" width="0.1524" layer="91"/>
+</segment>
+<segment>
+<pinref part="CON1" gate="G$1" pin="8"/>
+<wire x1="35.56" y1="180.34" x2="22.86" y2="180.34" width="0.1524" layer="91"/>
+<wire x1="22.86" y1="180.34" x2="22.86" y2="182.88" width="0.1524" layer="91"/>
+<pinref part="P+4" gate="VCC" pin="VCC"/>
+</segment>
+</net>

Commit message: fixing points added, overall pcb width modified, cable connections changed
Parts:
- J1, J2, J3, J4: device SparkFun-Connectors:CONN_05 -> custom:CONN_05
Connections:
- net GND: now also U$6.EN, U$6.OUT; no longer U$6.GND, U$6.IN
- net M_DIR1: now also CON1.4; no longer CON1.3
- net M_M0: now also CON1.5; no longer CON1.6
- net M_M1: now also CON1.3; no longer CON1.2
- net M_M2: now also CON1.1; no longer CON1.4
- net M_STEP1: now also CON1.2; no longer CON1.1
- net M_STEP2: now also CON1.6; no longer CON1.5
- net VBAT: now also U$6.GND; no longer U$6.EN
- net VCC: now also U$6.IN; no longer U$6.OUT
